File: pcb_ads1115/pcb_ads1115.kicad_pcb (KiCad board)
At the start: 2 copper layers, 93.5 x 41.9 mm, 12 parts, among them J1 CONN_01X03, J2 CONN_01X03, J3 CONN_01X03, J4 CONN_01X03, J5 CONN_01X10, J6 CONN_01X10, P1 CONN_01X04, P2 CONN_01X04

Commit message: update ADC card
Parts:
- removed REF01, REF02, REF03, REF04: MountingHole_3mm, Mounting_Holes:MountingHole_3mm
- J5, J6: footprint w_pin_strip:pin_socket_10 -> w_pin_strip:pin_strip_10
