File: Esp-12F/Esp-12F.kicad_pcb (KiCad board)
At the start: 2 copper layers, 19 parts, among them J1 UART, SW1 RST, SW2 SW_Push, U1 ESP-12F, U2 AMS1117-3.3

Commit message: Expansion usb
Parts:
- moved C4 73.7 mm to (119.2, 82.1), turned to 270 degrees
- moved C5 14.4 mm to (122.5, 82.1), turned to 270 degrees
- moved C3 12.8 mm to (112.5, 75.7), turned to 180 degrees
Changed lines of the file:
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@@
   )
   (module Capacitors_SMD:C_1206_HandSoldering (layer F.Cu)
-    (at 121.2215 85.0138 270)
+    (at 112.4712 75.692 180)
     (descr "Capacitor SMD 1206, hand soldering")
     (tags "capacitor 1206")
     (attr smd)
-    (fp_text reference C3 (at 0 -1.75 270) (layer F.SilkS)
+    (fp_text reference C3 (at 0 -1.75 180) (layer F.SilkS)
       (effects (font (size 1 1) (thickness 0.15)))
     )
-    (fp_text value 1uF (at 0 2 270) (layer F.Fab)
+    (fp_text value 1uF (at 0 2 180) (layer F.Fab)
+      (effects (font (size 1 1) (thickness 0.15)))
+    )
+    (fp_line (start 3.25 1.05) (end -3.25 1.05) (layer F.CrtYd) (width 0.05))
+    (fp_line (start 3.25 1.05) (end 3.25 -1.05) (layer F.CrtYd) (width 0.05))
+    (fp_line (start -3.25 -1.05) (end -3.25 1.05) (layer F.CrtYd) (width 0.05))
+    (fp_line (start -3.25 -1.05) (end 3.25 -1.05) (layer F.CrtYd) (width 0.05))
+    (fp_line (start -1 1.02) (end 1 1.02) (layer F.SilkS) (width 0.12))
+    (fp_line (start 1 -1.02) (end -1 -1.02) (layer F.SilkS) (width 0.12))
+    (fp_line (start -1.6 -0.8) (end 1.6 -0.8) (layer F.Fab) (width 0.1))
+    (fp_line (start 1.6 -0.8) (end 1.6 0.8) (layer F.Fab) (width 0.1))
+    (fp_line (start 1.6 0.8) (end -1.6 0.8) (layer F.Fab) (width 0.1))
+    (fp_line (start -1.6 0.8) (end -1.6 -0.8) (layer F.Fab) (width 0.1))
+    (fp_text user %R (at 0 -1.75 180) (layer F.Fab)
+      (effects (font (size 1 1) (thickness 0.15)))
+    )
+    (pad 2 smd rect (at 2 0 180) (size 2 1.6) (layers F.Cu F.Paste F.Mask)
+      (net 1 GND))
+    (pad 1 smd rect (at -2 0 180) (size 2 1.6) (layers F.Cu F.Paste F.Mask)
+      (net 4 +5V))
+    (model Capacitors_SMD.3dshapes/C_1206.wrl
+      (at (xyz 0 0 0))
+      (scale (xyz 1 1 1))
+      (rotate (xyz 0 0 0))
+    )
+  )
+  (module Capacitors_SMD:C_1206_HandSoldering (layer F.Cu)
+    (at 119.1768 82.1436 270)
+    (descr "Capacitor SMD 1206, hand soldering")
+    (tags "capacitor 1206")
+    (attr smd)
+    (fp_text reference C4 (at 0 -1.75 270) (layer F.SilkS)
+      (effects (font (size 1 1) (thickness 0.15)))
+    )
+    (fp_text value 10uF (at 0 2 270) (layer F.Fab)
       (effects (font (size 1 1) (thickness 0.15)))
     )
@@
       (net 1 GND))
     (pad 1 smd rect (at -2 0 270) (size 2 1.6) (layers F.Cu F.Paste F.Mask)
-      (net 4 +5V))
-    (model Capacitors_SMD.3dshapes/C_1206.wrl
-      (at (xyz 0 0 0))
-      (scale (xyz 1 1 1))
-      (rotate (xyz 0 0 0))
-    )
-  )
-  (module Capacitors_SMD:C_1206_HandSoldering (layer F.Cu)
-    (at 188.881 58.2676)
-    (descr "Capacitor SMD 1206, hand soldering")
-    (tags "capacitor 1206")
-    (attr smd)
-    (fp_text reference C4 (at 0 -1.75) (layer F.SilkS)
-      (effects (font (size 1 1) (thickness 0.15)))
-    )
-    (fp_text value 10uF (at 0 2) (layer F.Fab)
-      (effects (font (size 1 1) (thickness 0.15)))
-    )
-    (fp_line (start 3.25 1.05) (end -3.25 1.05) (layer F.CrtYd) (width 0.05))
-    (fp_line (start 3.25 1.05) (end 3.25 -1.05) (layer F.CrtYd) (width 0.05))
-    (fp_line (start -3.25 -1.05) (end -3.25 1.05) (layer F.CrtYd) (width 0.05))
-    (fp_line (start -3.25 -1.05) (end 3.25 -1.05) (layer F.CrtYd) (width 0.05))
-    (fp_line (start -1 1.02) (end 1 1.02) (layer F.SilkS) (width 0.12))
-    (fp_line (start 1 -1.02) (end -1 -1.02) (layer F.SilkS) (width 0.12))
-    (fp_line (start -1.6 -0.8) (end 1.6 -0.8) (layer F.Fab) (width 0.1))
-    (fp_line (start 1.6 -0.8) (end 1.6 0.8) (layer F.Fab) (width 0.1))
-    (fp_line (start 1.6 0.8) (end -1.6 0.8) (layer F.Fab) (width 0.1))
-    (fp_line (start -1.6 0.8) (end -1.6 -0.8) (layer F.Fab) (width 0.1))
-    (fp_text user %R (at 0 -1.75) (layer F.Fab)
-      (effects (font (size 1 1) (thickness 0.15)))
-    )
-    (pad 2 smd rect (at 2 0) (size 2 1.6) (layers F.Cu F.Paste F.Mask)
-      (net 1 GND))
-    (pad 1 smd rect (at -2 0) (size 2 1.6) (layers F.Cu F.Paste F.Mask)
       (net 3 +3V3))
     (model Capacitors_SMD.3dshapes/C_1206.wrl
@@
   )
   (module Capacitors_SMD:C_1206_HandSoldering (layer F.Cu)
-    (at 127.9078 95.5294)
+    (at 122.4788 82.1436 270)
     (descr "Capacitor SMD 1206, hand soldering")
     (tags "capacitor 1206")
     (attr smd)
-    (fp_text reference C5 (at 0 -1.75) (layer F.SilkS)
+    (fp_text reference C5 (at 0 -1.75 270) (layer F.SilkS)
       (effects (font (size 1 1) (thickness 0.15)))
     )
-    (fp_text value 470pF (at 0 2) (layer F.Fab)
+    (fp_text value 470pF (at 0 2 270) (layer F.Fab)
       (effects (font (size 1 1) (thickness 0.15)))
     )
-    (fp_text user %R (at 0 -1.75) (layer F.Fab)
+    (fp_text user %R (at 0 -1.75 270) (layer F.Fab)
       (effects (font (size 1 1) (thickness 0.15)))
     )
@@
     (fp_line (start 3.25 1.05) (end 3.25 -1.05) (layer F.CrtYd) (width 0.05))
     (fp_line (start 3.25 1.05) (end -3.25 1.05) (layer F.CrtYd) (width 0.05))
-    (pad 1 smd rect (at -2 0) (size 2 1.6) (layers F.Cu F.Paste F.Mask)
+    (pad 1 smd rect (at -2 0 270) (size 2 1.6) (layers F.Cu F.Paste F.Mask)
       (net 3 +3V3))
-    (pad 2 smd rect (at 2 0) (size 2 1.6) (layers F.Cu F.Paste F.Mask)
+    (pad 2 smd rect (at 2 0 270) (size 2 1.6) (layers F.Cu F.Paste F.Mask)
       (net 1 GND))
     (model Capacitors_SMD.3dshapes/C_1206.wrl
