File: monitorIO/monitorIO.kicad_pcb (KiCad board)
At the start: 2 copper layers, 28.1 x 26.7 mm, 17 parts, among them J1 Conn_01x09_Female

Commit message: Monitor io
Parts:
- D1, D2, D3, D4, D5, D6, D7, D8: footprint w_smd_leds:Led_PLCC2_3528 -> LEDs:LED_0603
- R1, R2, R3, R4, R5, R6, R7, R8: moved to B.Cu
- moved D8 17.6 mm to (140.6, 96.5)
- moved D7 17.4 mm to (140.6, 94.0)
- moved D6 17.3 mm to (140.6, 91.4)
- moved D1 17.2 mm to (140.6, 78.7)
- moved D5 17.2 mm to (140.6, 88.9)
- moved D2 17.1 mm to (140.6, 81.3)
- moved D4 17.1 mm to (140.6, 86.4)
- moved D3 17.1 mm to (140.6, 83.8)
- moved R3 11.1 mm to (142.7, 83.8)
- moved R4 11.1 mm to (142.7, 86.4)
- moved R1 11.1 mm to (142.7, 78.7)
- moved R2 11.1 mm to (142.7, 81.3)
- moved R7 11.0 mm to (142.8, 94.0)
- moved R5 11.0 mm to (142.8, 88.9)
- moved R6 11.0 mm to (142.8, 91.5)
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Routing:
- net GND: track 55.1 -> 25.7 mm, vias 1 -> 0
- net Net-(J1-Pad4): track 14.8 -> 2.54 mm
- net Net-(J1-Pad3): track 14.8 -> 2.54 mm
- net Net-(J1-Pad2): track 14.8 -> 2.54 mm
- net Net-(J1-Pad1): track 14.8 -> 2.54 mm
- net Net-(J1-Pad7): track 14.7 -> 2.55 mm
- net Net-(J1-Pad8): track 14.7 -> 2.55 mm
- net Net-(J1-Pad6): track 14.7 -> 2.55 mm
- net Net-(J1-Pad5): track 14.7 -> 2.55 mm
- net Net-(D8-Pad2): track 6.52 -> 2.10 mm, vias 0 -> 1
- net Net-(D7-Pad2): track 6.20 -> 2.12 mm, vias 0 -> 1
- net Net-(D1-Pad2): track 6.45 -> 2.46 mm, vias 0 -> 1
- net Net-(D2-Pad2): track 6.13 -> 2.15 mm, vias 0 -> 1
- net Net-(D6-Pad2): track 5.88 -> 2.24 mm, vias 0 -> 1
- net Net-(D3-Pad2): track 5.80 -> 2.21 mm, vias 0 -> 1
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- added copper zone on F.Cu, net GND
Other:
- board size 28.1 x 26.7 mm -> 9.1 x 23.3 mm

Commit message: changes in monitor led
Parts:
- moved D1 1.27 mm to (141.9, 78.7)
- moved D2 1.27 mm to (141.9, 81.3)
- moved D3 1.27 mm to (141.9, 83.8)
- moved D4 1.27 mm to (141.9, 86.4)
- moved D5 1.27 mm to (141.9, 88.9)
- moved D6 1.27 mm to (141.9, 91.4)
- moved D7 1.27 mm to (141.9, 94.0)
- moved D8 1.27 mm to (141.9, 96.5)
- moved R1 0.13 mm to (142.6, 78.7)
- moved R2 0.13 mm to (142.6, 81.3)
- moved R3 0.13 mm to (142.6, 83.8)
- moved R4 0.13 mm to (142.6, 86.4)
- moved R5 0.13 mm to (142.6, 88.9)
- moved R6 0.13 mm to (142.6, 91.5)
- moved R7 0.13 mm to (142.6, 94.0)
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Routing:
- net Net-(D2-Pad2): track 2.15 -> 7.44 mm
- net Net-(D5-Pad2): track 2.26 -> 7.29 mm
- net Net-(D8-Pad2): track 2.10 -> 3.06 mm
- net Net-(D7-Pad2): track 2.12 -> 3.04 mm
- net Net-(D6-Pad2): track 2.24 -> 3.12 mm
- net Net-(D3-Pad2): track 2.21 -> 3.10 mm
- net GND: track 25.7 -> 24.9 mm
- net Net-(D1-Pad2): track 2.46 -> 3.10 mm
- net Net-(D4-Pad2): track 2.50 -> 3.10 mm
Other:
- board size 9.1 x 23.3 mm -> 7.8 x 23.3 mm
- net class Default: trace_width 0.5 -> 0.25
- board text added: "WhatsApp 6677983021"
- board text added: "abeleduardo.hdz@gmail.com"
